File: GNERAL/GNERAL.kicad_sch (KiCad schematic)
At the start: 6 parts

Commit message: medio
Parts:
- added J?: Conn_01x05_Male, Connector_JST:JST_XH_B5B-XH-A_1x05_P2.50mm_Vertical, symbol Connector:Conn_01x05_Male
- added J?: Conn_01x05_Male, symbol Connector:Conn_01x05_Male
- R?: footprint (none) -> Resistor_SMD:R_0805_2012Metric_Pad1.20x1.40mm_HandSolder
Connections:
- net at R?.1: now also A?.21 (A2), J?.3 (Pin_3)
- net at R?.2: now also A?.24 (A5), A?.29 (GND), A?.4 (GND), R?.2, R?.2, R?.2, R?.2
- net at R?.1: now also A?.19 (A0), J?.1 (Pin_1)
- net at R?.1: now also A?.20 (A1), J?.2 (Pin_2)
- net at A?.22 (A3): now also R?.1, J?.4 (Pin_4)
- net at A?.23 (A4): now also R?.1, J?.5 (Pin_5)
- net at A?.27 (+5V): now also J?.1 (Pin_1), J?.2 (Pin_2), J?.3 (Pin_3), J?.4 (Pin_4), J?.5 (Pin_5)
- no-connect marks 0 -> 12
Other:
- moved on the sheet: R?

Commit message: hola
Parts:
- added J?: Conn_01x08_Female, Connector_PinSocket_2.54mm:PinSocket_1x08_P2.54mm_Vertical, symbol Connector:Conn_01x08_Female
- R1, R2, R3, R4, R5: renamed from R?; value R -> 220
- VDD1: renamed from J?; footprint (none) -> Connector_JST:JST_XH_B5B-XH-A_1x05_P2.50mm_Vertical
- gave numbers to parts that had none: 2
Connections:
- net at A1.29 (GND), R1.2, R2.2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: now also J?.2 (Pin_2); no longer A1.24 (A5), A1.4 (GND)
- net at A1.17 (3V3): now also J?.1 (Pin_1)
- net at A1.25 (A6): now also J?.4 (Pin_4)
- new net: A1.24 (A5), J?.3 (Pin_3)
- no-connect marks 12 -> 24

Commit message: c
Parts:
- removed J?: Conn_01x08_Female, Connector_PinSocket_2.54mm:PinSocket_1x08_P2.54mm_Vertical, symbol Connector:Conn_01x08_Female
- added J1: Conn_01x08_Female, Connector_PinSocket_2.54mm:PinSocket_1x08_P2.54mm_Vertical, symbol Connector:Conn_01x08_Female
- Data1: footprint Connector_JST:JST_XH_B5B-XH-A_1x05_P2.50mm_Vertical -> Connector_JST:JST_XH_S5B-XH-A-1_1x05_P2.50mm_Horizontal
- VDD1: footprint Connector_JST:JST_XH_B5B-XH-A_1x05_P2.50mm_Vertical -> Connector_JST:JST_XH_S5B-XH-A_1x05_P2.50mm_Horizontal
Connections:
- net at A1.29 (GND), R1.2, R2.2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: now also J1.2 (Pin_2)
- net at A1.17 (3V3): now also J1.1 (Pin_1)
- net at A1.24 (A5): now also J1.3 (Pin_3)
- net at A1.25 (A6): now also J1.4 (Pin_4)
Changed lines of the file:
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@@
     (pin "2")
+  )
+  (symbol (lib_id "Connector:Conn_01x05_Male") (at 191.77 86.36 0) (mirror y) (unit 1)
+    (in_bom yes) (on_board yes) (fields_autoplaced)
+    (property "Reference" "Data1" (id 0) (at 193.04 85.0899 0)
+      (effects (font (size 1.27 1.27)) (justify right))
+    )
+    (property "Value" "Conn_01x05_Male" (id 1) (at 193.04 87.6299 0)
+      (effects (font (size 1.27 1.27)) (justify right))
+    )
+    (property "Footprint" "Connector_JST:JST_XH_S5B-XH-A-1_1x05_P2.50mm_Horizontal" (id 2) (at 191.77 86.36 0)
+      (effects (font (size 1.27 1.27)) hide)
+    )
+    (property "Datasheet" "~" (id 3) (at 191.77 86.36 0)
+      (effects (font (size 1.27 1.27)) hide)
+    )
+    (pin "1")
+    (pin "2")
+    (pin "3")
+    (pin "4")
+    (pin "5")
   )
   (symbol (lib_id "Connector:Conn_01x08_Female") (at 68.58 64.77 0) (mirror y) (unit 1)
     (in_bom yes) (on_board yes) (fields_autoplaced)
-    (property "Reference" "J?" (id 0) (at 69.215 52.07 0))
+    (property "Reference" "J1" (id 0) (at 69.215 52.07 0))
     (property "Value" "Conn_01x08_Female" (id 1) (at 69.215 54.61 0))
-    (property "Footprint" "Connector_PinSocket_2.54mm:PinSocket_1x08_P2.54mm_Vertical" (id 2) (at 72.39 78.74 0)
+    (property "Footprint" "Connector_PinSocket_2.54mm:PinSocket_1x08_P2.54mm_Vertical" (id 2) (at 68.58 64.77 0)
       (effects (font (size 1.27 1.27)) hide)
     )
@@
     (pin "8")
   )
-  (symbol (lib_id "Connector:Conn_01x05_Male") (at 191.77 86.36 0) (mirror y) (unit 1)
-    (in_bom yes) (on_board yes) (fields_autoplaced)
-    (property "Reference" "Data1" (id 0) (at 193.04 85.0899 0)
-      (effects (font (size 1.27 1.27)) (justify right))
-    )
-    (property "Value" "Conn_01x05_Male" (id 1) (at 193.04 87.6299 0)
-      (effects (font (size 1.27 1.27)) (justify right))
-    )
-    (property "Footprint" "Connector_JST:JST_XH_B5B-XH-A_1x05_P2.50mm_Vertical" (id 2) (at 191.77 86.36 0)
-      (effects (font (size 1.27 1.27)) hide)
-    )
-    (property "Datasheet" "~" (id 3) (at 191.77 86.36 0)
-      (effects (font (size 1.27 1.27)) hide)
-    )
-    (pin "1")
-    (pin "2")
-    (pin "3")
-    (pin "4")
-    (pin "5")
-  )
   (symbol (lib_id "Connector:Conn_01x05_Male") (at 191.77 72.39 0) (mirror y) (unit 1)
     (in_bom yes) (on_board yes) (fields_autoplaced)
@@
       (effects (font (size 1.27 1.27)) (justify right))
     )
-    (property "Footprint" "Connector_JST:JST_XH_B5B-XH-A_1x05_P2.50mm_Vertical" (id 2) (at 191.77 72.39 0)
+    (property "Footprint" "Connector_JST:JST_XH_S5B-XH-A_1x05_P2.50mm_Horizontal" (id 2) (at 191.77 72.39 0)
       (effects (font (size 1.27 1.27)) hide)
     )
@@
     )
     (path "/79810072-220c-4855-8ed3-35508f1c9d6c"
-      (reference "Data1") (unit 1) (value "Conn_01x05_Male") (footprint "Connector_JST:JST_XH_B5B-XH-A_1x05_P2.50mm_Vertical")
+      (reference "Data1") (unit 1) (value "Conn_01x05_Male") (footprint "Connector_JST:JST_XH_S5B-XH-A-1_1x05_P2.50mm_Horizontal")
     )
-    (path "/784d6562-e40b-4397-9860-1c7951faa834"
-      (reference "J?") (unit 1) (value "Conn_01x08_Female") (footprint "Connector_PinSocket_2.54mm:PinSocket_1x08_P2.54mm_Vertical")
+    (path "/a43e9513-0378-4682-ae9a-858c99187627"
+      (reference "J1") (unit 1) (value "Conn_01x08_Female") (footprint "Connector_PinSocket_2.54mm:PinSocket_1x08_P2.54mm_Vertical")
     )
     (path "/e778434c-70bb-43a3-8d61-1c819198bab2"
@@
     )
     (path "/b46f5e0a-30c1-4d4d-a59a-f36ddee6a8ba"
-      (reference "VDD1") (unit 1) (value "Conn_01x05_Male") (footprint "Connector_JST:JST_XH_B5B-XH-A_1x05_P2.50mm_Vertical")
+      (reference "VDD1") (unit 1) (value "Conn_01x05_Male") (footprint "Connector_JST:JST_XH_S5B-XH-A_1x05_P2.50mm_Horizontal")
     )
   )

Commit message: requieroruteo
Parts:
- VDD1: footprint Connector_JST:JST_XH_S5B-XH-A_1x05_P2.50mm_Horizontal -> Connector_JST:JST_XH_S5B-XH-A-1_1x05_P2.50mm_Horizontal
Changed lines of the file:
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@@
       (effects (font (size 1.27 1.27)) (justify right))
     )
-    (property "Footprint" "Connector_JST:JST_XH_S5B-XH-A_1x05_P2.50mm_Horizontal" (id 2) (at 191.77 72.39 0)
+    (property "Footprint" "Connector_JST:JST_XH_S5B-XH-A-1_1x05_P2.50mm_Horizontal" (id 2) (at 191.77 72.39 0)
       (effects (font (size 1.27 1.27)) hide)
     )
@@
     )
     (path "/b46f5e0a-30c1-4d4d-a59a-f36ddee6a8ba"
-      (reference "VDD1") (unit 1) (value "Conn_01x05_Male") (footprint "Connector_JST:JST_XH_S5B-XH-A_1x05_P2.50mm_Horizontal")
+      (reference "VDD1") (unit 1) (value "Conn_01x05_Male") (footprint "Connector_JST:JST_XH_S5B-XH-A-1_1x05_P2.50mm_Horizontal")
     )
   )

Commit message: me canseee
Connections:
- net GND: now reaches A1.29 (GND), J1.2 (Pin_2), R1.2, R2.2, R3.2, R4.2, R5.2
Changed lines of the file:
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@@
   (junction (at 182.88 69.85) (diameter 0) (color 0 0 0 0)
   )
-  (junction (at 172.72 100.33) (diameter 0) (color 0 0 0 0)
-  )
   (junction (at 165.1 100.33) (diameter 0) (color 0 0 0 0)
   )
@@
   (junction (at 162.56 93.98) (diameter 0) (color 0 0 0 0)
   )
-  (junction (at 161.29 123.19) (diameter 0) (color 0 0 0 0)
-  )
-  (junction (at 172.72 92.71) (diameter 0) (color 0 0 0 0)
-  )
   (junction (at 182.88 63.5) (diameter 0) (color 0 0 0 0)
   )
@@
   )
   (junction (at 154.94 114.3) (diameter 0) (color 0 0 0 0)
-  )
-  (junction (at 127 123.19) (diameter 0) (color 0 0 0 0)
-  )
-  (junction (at 172.72 81.28) (diameter 0) (color 0 0 0 0)
   )
   (no_connect (at 111.76 86.36))
@@
     (stroke (width 0) (type default) (color 0 0 0 0))
   )
-  (wire (pts (xy 127 123.19) (xy 161.29 123.19))
-    (stroke (width 0) (type default) (color 0 0 0 0))
-  )
   (wire (pts (xy 73.66 64.77) (xy 90.17 64.77))
     (stroke (width 0) (type default) (color 0 0 0 0))
   )
-  (wire (pts (xy 172.72 81.28) (xy 172.72 92.71))
-    (stroke (width 0) (type default) (color 0 0 0 0))
-  )
-  (wire (pts (xy 172.72 100.33) (xy 172.72 123.19))
-    (stroke (width 0) (type default) (color 0 0 0 0))
-  )
   (wire (pts (xy 186.69 81.28) (xy 176.53 81.28))
     (stroke (width 0) (type default) (color 0 0 0 0))
@@
     (stroke (width 0) (type default) (color 0 0 0 0))
   )
-  (wire (pts (xy 127 114.3) (xy 127 123.19))
-    (stroke (width 0) (type default) (color 0 0 0 0))
-  )
   (wire (pts (xy 158.75 74.93) (xy 161.29 74.93))
     (stroke (width 0) (type default) (color 0 0 0 0))
@@
     (stroke (width 0) (type default) (color 0 0 0 0))
   )
-  (wire (pts (xy 143.51 119.38) (xy 143.51 101.6))
+  (wire (pts (xy 143.51 123.19) (xy 143.51 101.6))
     (stroke (width 0) (type default) (color 0 0 0 0))
   )
@@
     (stroke (width 0) (type default) (color 0 0 0 0))
   )
-  (wire (pts (xy 87.63 119.38) (xy 143.51 119.38))
+  (wire (pts (xy 87.63 123.19) (xy 143.51 123.19))
     (stroke (width 0) (type default) (color 0 0 0 0))
   )
@@
     (stroke (width 0) (type default) (color 0 0 0 0))
   )
-  (wire (pts (xy 82.55 123.19) (xy 127 123.19))
-    (stroke (width 0) (type default) (color 0 0 0 0))
-  )
   (wire (pts (xy 182.88 72.39) (xy 182.88 69.85))
     (stroke (width 0) (type default) (color 0 0 0 0))
   )
-  (wire (pts (xy 172.72 123.19) (xy 161.29 123.19))
-    (stroke (width 0) (type default) (color 0 0 0 0))
-  )
   (wire (pts (xy 154.94 114.3) (xy 154.94 115.57))
     (stroke (width 0) (type default) (color 0 0 0 0))
   )
-  (wire (pts (xy 90.17 64.77) (xy 90.17 118.11))
+  (wire (pts (xy 90.17 64.77) (xy 90.17 121.92))
     (stroke (width 0) (type default) (color 0 0 0 0))
   )
@@
     (stroke (width 0) (type default) (color 0 0 0 0))
   )
-  (wire (pts (xy 172.72 74.93) (xy 172.72 81.28))
-    (stroke (width 0) (type default) (color 0 0 0 0))
-  )
   (wire (pts (xy 162.56 96.52) (xy 162.56 100.33))
     (stroke (width 0) (type default) (color 0 0 0 0))
@@
     (stroke (width 0) (type default) (color 0 0 0 0))
   )
-  (wire (pts (xy 90.17 118.11) (xy 139.7 118.11))
-    (stroke (width 0) (type default) (color 0 0 0 0))
-  )
-  (wire (pts (xy 82.55 59.69) (xy 82.55 123.19))
+  (wire (pts (xy 90.17 121.92) (xy 142.24 121.92))
     (stroke (width 0) (type default) (color 0 0 0 0))
   )
@@
     (stroke (width 0) (type default) (color 0 0 0 0))
   )
-  (wire (pts (xy 139.7 104.14) (xy 137.16 104.14))
+  (wire (pts (xy 142.24 104.14) (xy 137.16 104.14))
     (stroke (width 0) (type default) (color 0 0 0 0))
   )
@@
     (stroke (width 0) (type default) (color 0 0 0 0))
   )
-  (wire (pts (xy 139.7 104.14) (xy 139.7 118.11))
+  (wire (pts (xy 142.24 104.14) (xy 142.24 121.92))
     (stroke (width 0) (type default) (color 0 0 0 0))
   )
@@
     (stroke (width 0) (type default) (color 0 0 0 0))
   )
-  (wire (pts (xy 172.72 92.71) (xy 172.72 100.33))
-    (stroke (width 0) (type default) (color 0 0 0 0))
-  )
   (wire (pts (xy 168.91 74.93) (xy 172.72 74.93))
     (stroke (width 0) (type default) (color 0 0 0 0))
@@
     (stroke (width 0) (type default) (color 0 0 0 0))
   )
-  (wire (pts (xy 87.63 62.23) (xy 87.63 119.38))
+  (wire (pts (xy 87.63 62.23) (xy 87.63 123.19))
     (stroke (width 0) (type default) (color 0 0 0 0))
   )
@@
     (stroke (width 0) (type default) (color 0 0 0 0))
   )
-  (wire (pts (xy 73.66 59.69) (xy 82.55 59.69))
-    (stroke (width 0) (type default) (color 0 0 0 0))
+  (global_label "GND" (shape input) (at 172.72 81.28 0) (fields_autoplaced)
+    (effects (font (size 1.27 1.27)) (justify left))
+    (property "Intersheet References" "${INTERSHEET_REFS}" (id 0) (at 179.0036 81.2006 0)
+      (effects (font (size 1.27 1.27)) (justify left) hide)
+    )
+  )
+  (global_label "GND" (shape input) (at 73.66 59.69 0) (fields_autoplaced)
+    (effects (font (size 1.27 1.27)) (justify left))
+    (property "Intersheet References" "${INTERSHEET_REFS}" (id 0) (at 79.9436 59.6106 0)
+      (effects (font (size 1.27 1.27)) (justify left) hide)
+    )
+  )
+  (global_label "GND" (shape input) (at 161.29 123.19 0) (fields_autoplaced)
+    (effects (font (size 1.27 1.27)) (justify left))
+    (property "Intersheet References" "${INTERSHEET_REFS}" (id 0) (at 167.5736 123.1106 0)
+      (effects (font (size 1.27 1.27)) (justify left) hide)
+    )
+  )
+  (global_label "GND" (shape input) (at 172.72 74.93 0) (fields_autoplaced)
+    (effects (font (size 1.27 1.27)) (justify left))
+    (property "Intersheet References" "${INTERSHEET_REFS}" (id 0) (at 179.0036 74.8506 0)
+      (effects (font (size 1.27 1.27)) (justify left) hide)
+    )
+  )
+  (global_label "GND" (shape input) (at 172.72 92.71 0) (fields_autoplaced)
+    (effects (font (size 1.27 1.27)) (justify left))
+    (property "Intersheet References" "${INTERSHEET_REFS}" (id 0) (at 179.0036 92.6306 0)
+      (effects (font (size 1.27 1.27)) (justify left) hide)
+    )
+  )
+  (global_label "GND" (shape input) (at 127 114.3 270) (fields_autoplaced)
+    (effects (font (size 1.27 1.27)) (justify right))
+    (property "Intersheet References" "${INTERSHEET_REFS}" (id 0) (at 127.0794 120.5836 90)
+      (effects (font (size 1.27 1.27)) (justify right) hide)
+    )
+  )
+  (global_label "GND" (shape input) (at 172.72 100.33 0) (fields_autoplaced)
+    (effects (font (size 1.27 1.27)) (justify left))
+    (property "Intersheet References" "${INTERSHEET_REFS}" (id 0) (at 179.0036 100.2506 0)
+      (effects (font (size 1.27 1.27)) (justify left) hide)
+    )
   )
   (symbol (lib_id "Device:R") (at 167.64 92.71 90) (unit 1)
