File: GNERAL/GNERAL.kicad_pcb (KiCad board)
At the start: 2 copper layers, 9 parts, among them J1 Conn_01x08_Female

Commit message: requieroruteo
Parts:
- VDD1: footprint Connector_JST:JST_XH_S5B-XH-A_1x05_P2.50mm_Horizontal -> Connector_JST:JST_XH_S5B-XH-A-1_1x05_P2.50mm_Horizontal
- moved VDD1 1.56 mm to (164.1, 85.7)
- moved R2 0.53 mm to (155.1, 106.5)
- moved R3 0.49 mm to (155.0, 101.8)
- moved R4 0.05 mm to (155.0, 97.3)

Commit message: me canseee
Parts:
- moved A1 0.05 mm to (146.8, 114.4)
Connections:
- net Net-(A1-Pad29) renamed GND
Routing:
- added copper zone on B.Cu, net (none)
- added copper zone on F.Cu, net (none)
Other:
- board outline added: 43.7 x 49.7 mm
Changed lines of the file:
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@@
   (net 27 "Net-(A1-Pad27)")
   (net 28 "unconnected-(A1-Pad28)")
-  (net 29 "Net-(A1-Pad29)")
+  (net 29 "GND")
   (net 30 "unconnected-(A1-Pad30)")
   (net 31 "unconnected-(J1-Pad5)")
@@
       (net 22 "Net-(A1-Pad22)") (pintype "passive"))
     (pad "2" smd roundrect (at 1 0) (size 1.2 1.4) (layers "F.Cu" "F.Paste" "F.Mask") (roundrect_rratio 0.208333)
-      (net 29 "Net-(A1-Pad29)") (pintype "passive"))
+      (net 29 "GND") (pintype "passive"))
     (model "${KICAD6_3DMODEL_DIR}/Resistor_SMD.3dshapes/R_0805_2012Metric.wrl"
       (offset (xyz 0 0 0))
@@
   )
   (footprint "Module:Arduino_Nano" (layer "F.Cu")
-    (at 146.82 114.43 180)
+    (at 146.81 114.38 180)
     (descr "Arduino Nano, http://www.mouser.com/pdfdocs/Gravitech_Arduino_Nano3_0.pdf")
     (tags "Arduino Nano")
@@
       (net 28 "unconnected-(A1-Pad28)") (pinfunction "~{RESET}") (pintype "input+no_connect"))
     (pad "29" thru_hole oval (at 15.24 2.54 180) (size 1.6 1.6) (drill 1) (layers *.Cu *.Mask)
-      (net 29 "Net-(A1-Pad29)") (pinfunction "GND") (pintype "power_out"))
+      (net 29 "GND") (pinfunction "GND") (pintype "power_out"))
     (pad "30" thru_hole oval (at 15.24 0 180) (size 1.6 1.6) (drill 1) (layers *.Cu *.Mask)
       (net 30 "unconnected-(A1-Pad30)") (pinfunction "VIN") (pintype "power_in+no_connect"))
@@
       (net 21 "Net-(A1-Pad21)") (pintype "passive"))
     (pad "2" smd roundrect (at 1 0) (size 1.2 1.4) (layers "F.Cu" "F.Paste" "F.Mask") (roundrect_rratio 0.208333)
-      (net 29 "Net-(A1-Pad29)") (pintype "passive"))
+      (net 29 "GND") (pintype "passive"))
     (model "${KICAD6_3DMODEL_DIR}/Resistor_SMD.3dshapes/R_0805_2012Metric.wrl"
       (offset (xyz 0 0 0))
@@
       (net 23 "Net-(A1-Pad23)") (pintype "passive"))
     (pad "2" smd roundrect (at 1 0) (size 1.2 1.4) (layers "F.Cu" "F.Paste" "F.Mask") (roundrect_rratio 0.208333)
-      (net 29 "Net-(A1-Pad29)") (pintype "passive"))
+      (net 29 "GND") (pintype "passive"))
     (model "${KICAD6_3DMODEL_DIR}/Resistor_SMD.3dshapes/R_0805_2012Metric.wrl"
       (offset (xyz 0 0 0))
@@
     (property "Sheetname" "")
     (attr through_hole)
-    (fp_text reference "J1" (at 0 -2.77 90) (layer "F.SilkS")
+    (fp_text reference "J1" (at 3.02 0.99 90) (layer "F.SilkS")
       (effects (font (size 1 1) (thickness 0.15)))
     )
@@
       (net 17 "Net-(A1-Pad17)") (pinfunction "Pin_1") (pintype "passive"))
     (pad "2" thru_hole oval (at 0 2.54 270) (size 1.7 1.7) (drill 1) (layers *.Cu *.Mask)
-      (net 29 "Net-(A1-Pad29)") (pinfunction "Pin_2") (pintype "passive"))
+      (net 29 "GND") (pinfunction "Pin_2") (pintype "passive"))
     (pad "3" thru_hole oval (at 0 5.08 270) (size 1.7 1.7) (drill 1) (layers *.Cu *.Mask)
       (net 24 "Net-(A1-Pad24)") (pinfunction "Pin_3") (pintype "passive"))
@@
       (net 19 "Net-(A1-Pad19)") (pintype "passive"))
     (pad "2" smd roundrect (at 1 0 180) (size 1.2 1.4) (layers "F.Cu" "F.Paste" "F.Mask") (roundrect_rratio 0.208333)
-      (net 29 "Net-(A1-Pad29)") (pintype "passive"))
+      (net 29 "GND") (pintype "passive"))
     (model "${KICAD6_3DMODEL_DIR}/Resistor_SMD.3dshapes/R_0805_2012Metric.wrl"
       (offset (xyz 0 0 0))
@@
     (property "Sheetname" "")
     (attr through_hole)
-    (fp_text reference "VDD1" (at 5 -5.1 90) (layer "F.SilkS")
-      (effects (font (size 1 1) (thickness 0.15)))
-    )
-    (fp_text value "Conn_01x05_Male" (at 5 8.8 90) (layer "F.Fab")
+    (fp_text reference "VDD1" (at 5.17 -2.84 90) (layer "F.SilkS")
+      (effects (font (size 1 1) (thickness 0.15)))
+    )
+    (fp_text value "Conn_01x05_Male" (at 5.31 4.64 90) (layer "F.Fab")
       (effects (font (size 1 1) (thickness 0.15)))
     )
@@
       (net 20 "Net-(A1-Pad20)") (pintype "passive"))
     (pad "2" smd roundrect (at 1 0) (size 1.2 1.4) (layers "F.Cu" "F.Paste" "F.Mask") (roundrect_rratio 0.208333)
-      (net 29 "Net-(A1-Pad29)") (pintype "passive"))
+      (net 29 "GND") (pintype "passive"))
     (model "${KICAD6_3DMODEL_DIR}/Resistor_SMD.3dshapes/R_0805_2012Metric.wrl"
       (offset (xyz 0 0 0))
@@
       (effects (font (size 1 1) (thickness 0.15)))
     )
-    (fp_text value "Conn_01x05_Male" (at 5 8.8 90) (layer "F.Fab")
+    (fp_text value "Conn_01x05_Male" (at 3.27 4.65 90) (layer "F.Fab")
       (effects (font (size 1 1) (thickness 0.15)))
     )
@@
     )
   )
-  (gr_rect (start 128.85 71.31) (end 172.98 121.53) (layer "F.Cu") (width 0.2) (fill none))
+  (gr_rect (start 129.12 71.54) (end 172.78 121.25) (layer "Edge.Cuts") (width 0.1) (fill none))
+  (zone (net 0) (net_name "") (layers F&B.Cu) (hatch edge 0.508)
+    (connect_pads (clearance 0.508))
+    (min_thickness 0.254) (filled_areas_thickness no)
+    (fill yes (thermal_gap 0.508) (thermal_bridge_width 0.508))
+    (polygon
+      (pts
+        (xy 172.7 121.3)
+        (xy 129.1 121.3)
+        (xy 129.11 71.6)
+        (xy 172.8 71.5)
+      )
+    )
+  )
 )

Commit message: FNIAL
Parts:
- added KL: LOGO, lgoooo:logod, F.Cu at (155.3, 79.8)
Routing:
- net GND: track 0.00 -> 69.2 mm
- net Net-(A1-Pad27): track 0.00 -> 62.3 mm
- net Net-(A1-Pad17): track 0.00 -> 60.1 mm
- net Net-(A1-Pad19): track 0.00 -> 55.6 mm
- net Net-(A1-Pad21): track 0.00 -> 54.9 mm
- net Net-(A1-Pad20): track 0.00 -> 53.6 mm
- net Net-(A1-Pad22): track 0.00 -> 44.5 mm
- net Net-(A1-Pad23): track 0.00 -> 39.3 mm
- net Net-(A1-Pad24): track 0.00 -> 39.1 mm
- net Net-(A1-Pad25): track 0.00 -> 35.5 mm
Other:
- board text added: "DR-JD"
